Commit message: Update model  and control.

File: robot_model.urdf (robot description, URDF)
Before this commit: robot rc_rover_arm, 12 links, 11 joints
Links:
- removed link forearm_roll_link
Joints:
- removed joint forearm_roll_joint
- joint wrist_pitch_joint: origin xyz=0 0 0.04 rpy=0 0 0 -> xyz=0 0 0.08 rpy=0 0 0; parent forearm_roll_link -> elbow_link
